File: Kicad Files/Mainpcb.kicad_pcb (KiCad board)
At the start: 2 copper layers, 257.2 x 100 mm, 144 parts, among them SW1 SW_Push, SW2 Rotary_Encoder_Switch, U1 ProMicro

Commit message: a
Parts:
- moved D_53 14.3 mm to (173.8, 111.9)
- moved D_48 6.74 mm to (59.5, 116.7)
- moved D_50 4.76 mm to (92.9, 116.7)
- moved D_52 4.76 mm to (131.0, 116.7)
- moved D_55 4.76 mm to (207.2, 116.7)
- moved D_57 4.76 mm to (245.3, 116.7)
- moved D_0 4.76 mm to (54.8, 40.5)
- moved D_10 4.76 mm to (245.3, 40.5)
- moved D_2 4.76 mm to (92.9, 40.5)
- moved D_36 4.76 mm to (54.8, 97.6)
- moved D_38 4.76 mm to (92.9, 97.6)
- moved D_4 4.76 mm to (131.0, 40.5)
- moved D_40 4.76 mm to (131.0, 97.6)
- moved D_42 4.76 mm to (169.1, 97.6)
- moved D_44 4.76 mm to (207.2, 97.6)
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Routing:
- net col5: track 390.6 -> 502.3 mm, vias 1 -> 0
- net col2: track 300.1 -> 394.5 mm
- net GND: track 70.6 -> 0.00 mm
- net Net-(D_53-Pad2): track 17.5 -> 31.2 mm
- net row1: track 257.1 -> 245.4 mm
- net row5: track 281.6 -> 272.1 mm
- net col0: track 205.4 -> 198.2 mm
- net row7: track 290.8 -> 285.5 mm
- net Net-(D_48-Pad2): track 17.5 -> 22.3 mm
- net row4: track 255.7 -> 260.1 mm
- net row6: track 264.6 -> 269.0 mm
- net row0: track 227.6 -> 224.9 mm
- net Net-(D_55-Pad2): track 15.5 -> 18.2 mm
- net Net-(D_57-Pad2): track 15.5 -> 18.2 mm
- net row2: track 222.5 -> 224.7 mm
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
Commit message: Fixed files and imroved pcb design
Parts:
- added REF**: Stabilizer_MX_2u, keyswitches:Stabilizer_MX_2u, F.Cu at (159.5, 107.2)
Routing:
- net col5: track 502.3 -> 387.9 mm, vias 0 -> 1
- net col2: track 394.5 -> 285.5 mm, vias 0 -> 1
- net row7: track 285.5 -> 289.3 mm
- net row8: track 280.8 -> 278.8 mm
- net col3: track 314.4 -> 316.2 mm
- net row0: track 224.9 -> 223.3 mm, vias 0 -> 1
- net row9: track 293.4 -> 294.8 mm
- net row4: track 260.1 -> 261.1 mm
- net col4: track 350.9 -> 351.8 mm
- net Net-(SW1-Pad1): track 57.9 -> 57.4 mm
