File: Kicad Files/bottom.kicad_pcb (KiCad board)
At the start: 2 copper layers, 257.2 x 100 mm, 18 parts

Commit message: Fixed files and imroved pcb design
Parts:
- added REF**: MountingHole_2.2mm_M2, MountingHole:MountingHole_2.2mm_M2, F.Cu at (197.6, 59.5)
- added REF**: MountingHole_2.2mm_M2, MountingHole:MountingHole_2.2mm_M2, F.Cu at (121.4, 59.5)
