File: Kicad Files/top.kicad_pcb (KiCad board)
At the start: 2 copper layers, 233.4 x 100 mm, 68 parts, among them SW2 KEY_SWITCH

Commit message: Fixed files and imroved pcb design
Parts:
- removed SW2 (x58): KEY_SWITCH, kbd:SW_Hole
Other:
- outline, holes or cut-outs redrawn
